Commit message: URDF Correction & Odom

File: Mobile_Robot/src/diff_drive_robot/description/robot_core.xacro (robot description, xacro)
@@ -4,27 +4,23 @@
   <xacro:property name="pi" value="3.14159265359"/>
   <xacro:include filename="inertial_macros.xacro"/>
-  <!-- Materials -->
-  <material name="white">
-    <color rgba="1 1 1 1"/>
-  </material>
-  <material name="orange">
-    <color rgba="1 0.3 0.1 1"/>
-  </material>
-  <material name="blue">
-    <color rgba="0.2 0.2 1 1"/>
-  </material>
-  <material name="black">
-    <color rgba="0 0 0 1"/>
-  </material>
+  <xacro:include filename="materials.xacro"/>
+  <xacro:include filename="gazebo.xacro"/>
+  <!-- Ground Reference -->
+    <link name="base_footprint"/>
+    <joint name="base_footprint_joint" type="fixed">
+        <parent link="base_footprint"/>
+        <child link="base_link"/>
+        <origin xyz="-0.1 0 0" rpy="0 0 0"/>
+    </joint>
   <!-- Base link -->
-  <link name="base_link">
-  </link>
+  <!-- <link name="base_link">
+  </link> -->
   <!-- Chassis link -->
-  <joint name="chassis_joint" type="fixed">
+  <!-- <joint name="chassis_joint" type="fixed">
     <parent link="base_link"/>
     <child link="chassis"/>
     <origin xyz="-0.1 0 0"/>
-  </joint>
-  <link name="chassis">
+  </joint> -->
+  <link name="base_link">
     <visual>
       <origin xyz="0.15 0 0.075"/>
@@ -46,51 +42,53 @@
   <!-- Left wheel -->
   <joint name="left_wheel_joint" type="continuous">
+        <parent link="base_link"/>
+        <child link="left_wheel"/>
+        <!-- Y = chassis_width/2 + wheel_thickness/2 = 0.15 + 0.02 = 0.17 -->
+        <origin xyz="0.1 0.17 0" rpy="-${pi/2} 0 0"/>
+        <axis xyz="0 0 1"/>
+    </joint>
+    <link name="left_wheel">
+        <visual>
+            <geometry>
+                <cylinder radius="0.05" length="0.04"/>
+            </geometry>
+            <material name="blue"/>
+        </visual>
+        <collision>
+            <geometry>
+                <cylinder radius="0.05" length="0.04"/>
+            </geometry>
+        </collision>
+        <xacro:inertial_cylinder mass="0.1" length="0.04" radius="0.05">
+            <origin xyz="0 0 0" rpy="0 0 0"/>
+        </xacro:inertial_cylinder>
+    </link>
+    <!-- Right wheel -->
+    <joint name="right_wheel_joint" type="continuous">
+        <parent link="base_link"/>
+        <child link="right_wheel"/>
+        <!-- Y = -(chassis_width/2 + wheel_thickness/2) = -0.17 -->
+        <origin xyz="0.1 -0.17 0" rpy="-${pi/2} 0 0"/>
+        <axis xyz="0 0 1"/>
+    </joint>
+    <link name="right_wheel">
+        <visual>
+            <geometry>
+                <cylinder radius="0.05" length="0.04"/>
+            </geometry>
+            <material name="blue"/>
+        </visual>
+        <collision>
+            <geometry>
+                <cylinder radius="0.05" length="0.04"/>
+            </geometry>
+        </collision>
+        <xacro:inertial_cylinder mass="0.1" length="0.04" radius="0.05">
+            <origin xyz="0 0 0" rpy="0 0 0"/>
+        </xacro:inertial_cylinder>
+    </link>
+  <!-- Caster wheel -->
+  <joint name="caster_wheel_joint" type="fixed">
     <parent link="base_link"/>
-    <child link="left_wheel"/>
-    <origin xyz="0 0.175 0" rpy="${pi/2} 0 0"/>
-    <axis xyz="0 0 1"/>
-  </joint>
-  <link name="left_wheel">
-    <visual>
-      <geometry>
-        <cylinder radius="0.05" length="0.04"/>
-      </geometry>
-      <material name="blue"/>
-    </visual>
-    <collision>
-        <geometry>
-            <cylinder radius="0.05" length="0.04"/>
-        </geometry>
-    </collision>
-    <xacro:inertial_cylinder mass="0.1" length="0.04" radius="0.05">
-        <origin xyz="0 0 0" rpy="0 0 0"/>
-    </xacro:inertial_cylinder>
-  </link>
-  <!-- Right wheel -->
-  <joint name="right_wheel_joint" type="continuous">
-    <parent link="base_link"/>
-    <child link="right_wheel"/>
-    <origin xyz="0 -0.175 0" rpy="${pi/2} 0 0"/>
-    <axis xyz="0 0 -1"/>
-  </joint>
-  <link name="right_wheel">
-    <visual>
-      <geometry>
-        <cylinder radius="0.05" length="0.04"/>
-      </geometry>
-      <material name="blue"/>
-    </visual>
-    <collision>
-        <geometry>
-            <cylinder radius="0.05" length="0.04"/>
-        </geometry>
-    </collision>
-    <xacro:inertial_cylinder mass="0.1" length="0.04" radius="0.05">
-        <origin xyz="0 0 0" rpy="0 0 0"/>
-    </xacro:inertial_cylinder>
-  </link>
-  <!-- Caster wheel -->
-  <joint name="caster_wheel_joint" type="continuous">
-    <parent link="chassis"/>
     <child link="caster_wheel"/>
     <origin xyz="0.24 0 0"/>
@@ -112,3 +110,10 @@
     </xacro:inertial_sphere>
   </link>
+  <!-- IMU -->
+  <link name="imu_frame"/>
+    <joint name="imu_joint" type="fixed">
+        <parent link="base_link"/>
+        <child link="imu_frame"/>
+        <origin xyz="0.0 0.0 0.08" rpy="0.0 0.0 0.0"/>
+    </joint>
 </robot>
