Commit message: Lidar IMU CAMERA ODOM Done

File: Mobile_Robot/src/diff_drive_robot/description/gazebo.xacro (robot description, xacro)
@@ -38,6 +38,11 @@
             <always_on>true</always_on>
             <update_rate>100</update_rate>
-            <topic>imu</topic>
-            <gz_frame_id>imu_frame</gz_frame_id>
+            <topic>/imu</topic>
+            <plugin filename="ignition-gazebo-imu-system" name="ignition::gazebo::systems::Imu">
+            <topic>/imu</topic>
+            <frame_id>imu_frame</frame_id>
+            <angular_velocity_noise>0.0002</angular_velocity_noise>
+            <linear_acceleration_noise>0.0002</linear_acceleration_noise>
+            </plugin>
         </sensor>
     </gazebo>

File: Mobile_Robot/src/diff_drive_robot/description/gz.xacro (robot description, xacro)
@@ -1,3 +1,3 @@
-<?xml version="1.0"?>
+<!-- <?xml version="1.0"?>
 <robot xmlns:xacro="http://www.ros.org/wiki/xacro">
     <!-- ........................... SENSOR PLUGIN ................................... -->
@@ -19,3 +19,3 @@
             <topic>imu</topic>
         </sensor>
-        </gazebo>
+        </gazebo> -->

File: Mobile_Robot/src/diff_drive_robot/description/robot_core.xacro (robot description, xacro)
@@ -110,10 +110,98 @@
     </xacro:inertial_sphere>
   </link>
+  <!-- Lidar -->
+  <joint name="laser_joint" type="fixed">
+        <parent link="base_link"/>
+        <child link="laser_frame"/>
+        <origin xyz="0.1 0 0.17" rpy="0 0 0"/>
+    </joint>
+    <link name="laser_frame">
+        <visual>
+            <geometry>
+                <cylinder radius="0.05" length="0.04"/>
+            </geometry>
+            <material name="red"/>
+        </visual>
+        <collision>
+            <geometry>
+                <cylinder radius="0.05" length="0.04"/>
+            </geometry>
+        </collision>
+        <xacro:inertial_cylinder mass="0.1" length="0.04" radius="0.05">
+            <origin xyz="0 0 0" rpy="0 0 0"/>
+        </xacro:inertial_cylinder>
+    </link>
+    <!-- Camera -->
+    <joint name="camera_joint" type="fixed">
+        <parent link="base_link"/>
+        <child link="camera_link"/>
+        <origin xyz="0.305 0 0.08" rpy="0 0 0"/>
+    </joint>
+    <link name="camera_link">
+        <visual>
+            <geometry>
+                <box size="0.010 0.03 0.03"/>
+            </geometry>
+            <material name="red"/>
+        </visual>
+    </link>
+    <joint name="camera_optical_joint" type="fixed">
+        <parent link="camera_link"/>
+        <child link="camera_link_optical"/>
+        <origin xyz="0 0 0" rpy="${-pi/2} 0 ${-pi/2}"/>
+    </joint>
+    <link name="camera_link_optical"></link>
+    <gazebo reference="camera_link">
+        <material>Gazebo/Red</material>
+        <sensor name="camera" type="camera">
+            <pose> 0 0 0 0 0 0 </pose>
+            <visualize>true</visualize>
+            <update_rate>10</update_rate>
+            <camera>
+                <camera_info_topic>camera/camera_info</camera_info_topic>
+                <horizontal_fov>1.089</horizontal_fov>
+                <image>
+                    <format>R8G8B8</format>
+                    <width>640</width>
+                    <height>480</height>
+                </image>
+                <clip>
+                    <near>0.05</near>
+                    <far>8.0</far>
+                </clip>
+            </camera>
+            <topic>camera/image_raw</topic>
+            <gz_frame_id>camera_link_optical</gz_frame_id>
+        </sensor>
+    </gazebo>
+    <gazebo reference="laser_frame">
+        <material>Gazebo/Red</material>
+        <sensor name="laser" type="gpu_lidar">
+            <pose> 0 0 0 0 0 0 </pose>
+            <visualize>true</visualize>
+            <update_rate>10</update_rate>
+            <lidar>
+                <scan>
+                    <horizontal>
+                        <samples>360</samples>
+                        <min_angle>-3.14</min_angle>
+                        <max_angle>3.14</max_angle>
+                    </horizontal>
+                </scan>
+                <range>
+                    <min>0.3</min>
+                    <max>12</max>
+                </range>
+            </lidar>
+            <topic>scan</topic>
+            <gz_frame_id>laser_frame</gz_frame_id>
+        </sensor>
+    </gazebo>
   <!-- IMU -->
   <link name="imu_frame"/>
     <joint name="imu_joint" type="fixed">
-        <parent link="base_link"/>
-        <child link="imu_frame"/>
-        <origin xyz="0.0 0.0 0.08" rpy="0.0 0.0 0.0"/>
+    <parent link="base_link"/>
+    <child link="imu_frame"/>
+    <origin xyz="0 0 0.08" rpy="0 0 0"/>
     </joint>
 </robot>
